Commit message: 现在能够在gazebo中进行仿真

File: install/moveit_resources_panda_description/share/moveit_resources_panda_description/urdf/panda.urdf (robot description, URDF)
Before this commit: robot panda, 12 links, 11 joints
Links:
- removed link panda_link8
- added link world
Joints:
- removed joint panda_joint8
- added joint world_joint: type fixed, parent world, child panda_link0, origin xyz=0 0 0 rpy=0 0 0
- joint panda_finger_joint2: mimic joint=panda_finger_joint1 -> (none)
- joint panda_hand_joint: origin xyz=0 0 0 rpy=0 0 -0.785398163397 -> xyz=0 0 0.107 rpy=0 0 -0.785398163397; parent panda_link8 -> panda_link7

File: install/panda_moveit_config/share/panda_moveit_config/config/panda.ros2_control.xacro (robot description, xacro)
@@ -2,5 +2,5 @@
 <robot xmlns:xacro="http://www.ros.org/wiki/xacro">
     <xacro:macro name="panda_ros2_control" params="name initial_positions_file">
-        <xacro:property name="initial_positions" value="${load_yaml(initial_positions_file)['initial_positions']}"/>
+        <xacro:property name="initial_positions" value="${xacro.load_yaml(initial_positions_file)['initial_positions']}"/>
         <ros2_control name="${name}" type="system">
             <hardware>

File: install/panda_moveit_config/share/panda_moveit_config/config/panda.urdf.xacro (robot description, xacro)
@@ -3,5 +3,5 @@
     <xacro:arg name="initial_positions_file" default="initial_positions.yaml" />
     <!-- Import panda urdf file -->
-    <xacro:include filename="$(find moveit_resources_panda_description)/urdf/panda.urdf" />
+    <xacro:include filename="$(find moveit_resources_panda_description)/urdf/panda.urdf.xacro" />
     <!-- Import control_xacro -->
     <xacro:include filename="panda.ros2_control.xacro" />

Commit message: 在gazebo中机械臂瘫在地上

File: install/moveit_resources_panda_description/share/moveit_resources_panda_description/urdf/panda.urdf (robot description, URDF)
Before this commit: robot panda, 12 links, 11 joints
Links:
- link panda_hand: mass None -> 0.5
- link panda_leftfinger: mass None -> 0.1
- link panda_link0: mass None -> 2.0
- link panda_link1: mass None -> 1.5
- link panda_link2: mass None -> 1.5
- link panda_link3: mass None -> 1.5
- link panda_link4: mass None -> 1.2
- link panda_link5: mass None -> 1.2
- link panda_link6: mass None -> 1.0
- link panda_link7: mass None -> 1.0
- link panda_rightfinger: mass None -> 0.1

File: install/panda_moveit_config/share/panda_moveit_config/config/panda.urdf.xacro (robot description, xacro)
@@ -6,4 +6,11 @@
     <!-- Import control_xacro -->
     <xacro:include filename="panda.ros2_control.xacro" />
+    <!-- Add a fixed joint to connect the robot to the world -->
+    <link name="world"/>
+    <joint name="world_joint" type="fixed">
+        <parent link="world"/>
+        <child link="panda_link0"/>
+        <origin xyz="0 0 0" rpy="0 0 0"/>
+    </joint>
     <xacro:panda_ros2_control name="FakeSystem" initial_positions_file="$(arg initial_positions_file)"/>
 </robot>
